Commit message: Correct position

File: src/manipulator1ver/urdf/links_joints.xacro (robot description, xacro)
@@ -62,5 +62,5 @@
     </link>
   </xacro:macro>
-  <xacro:macro name="m_link_mesh" params="name origin_xyz origin_rpy meshfile meshscale mass ixx ixy ixz iyy iyz izz">
+  <xacro:macro name="m_link_mesh" params="name origin_xyz origin_rpy meshfile meshscale mass ixx ixy ixz iyy iyz izz ">
     <link name="${name}">
       <inertial>
@@ -80,5 +80,5 @@
           <mesh filename="${meshfile}" scale="${meshscale}"/>
         </geometry>
-        <material name="light_black"/>
+        <material name="white"/>
       </visual>
     </link>

File: src/manipulator1ver/urdf/mrm.xacro (robot description, xacro)
@@ -5,7 +5,10 @@
   <xacro:include filename="$(find manipulator1ver)/urdf/links_joints.xacro" />
   <!-- END - Include -->
+    <material name="white">
+    <color rgba="1 1 1 1"/>
+  </material>
   <!-- BGN - Robot description -->
   <m_link_mesh name="${link_00_name}"
-              origin_rpy="0 0 0" origin_xyz="0 0 0"
+              origin_rpy="1.57 0 0" origin_xyz="0 0 0"
               mass="157.633"
               ixx="13.235" ixy="0" ixz="0"
@@ -13,12 +16,13 @@
               izz="9.655"
               meshfile="package://manipulator1ver/meshes/stl/1base.stl"
-              meshscale="0.001 0.001 0.001" />
+              meshscale="0.001 0.001 0.001"
+			  />
   <m_joint name="${link_00_name}__${link_01_name}" type="revolute"
            axis_xyz="0 0 1"
-           origin_rpy="0 0 0" origin_xyz="0 0 0.1"
+           origin_rpy="0 0 0" origin_xyz="0 0 0"
            parent="base_link" child="link_01"
            limit_e="1000" limit_l="-3.14" limit_u="3.14" limit_v="0.5" />
   <m_link_mesh name="${link_01_name}"
-              origin_rpy="0 0 0" origin_xyz="0 0 0.1"
+              origin_rpy="1.57 0 0" origin_xyz="0 0 0.0059"
               mass="157.633"
               ixx="13.235" ixy="0" ixz="0"
