Commit message: Karantin

File: src/manipulator1ver/urdf/mrm.xacro (robot description, xacro)
@@ -19,7 +19,7 @@
   <m_joint name="${link_00_name}__${link_01_name}" type="revolute"
            axis_xyz="0 0 1"
-           origin_rpy="0 0 0" origin_xyz="0 0 0.059"
+           origin_rpy="0 0 0" origin_xyz="0 0 0.0619"
            parent="base_link" child="link_01"
-           limit_e="1000" limit_l="-3.14" limit_u="3.14" limit_v="0.5" />
+           limit_e="1000" limit_l="-1.57" limit_u="1.57" limit_v="0.5" />
   <m_link_mesh name="${link_01_name}"
               origin_rpy="1.57 0 0" origin_xyz="0 0 0"
@@ -30,10 +30,10 @@
               meshfile="package://manipulator1ver/meshes/stl/2.stl"
               meshscale="0.001 0.001 0.001" />
-    <m_joint name="${link_01_name}__${link_02_name}" type="revolute"
+  <m_joint name="${link_01_name}__${link_02_name}" type="revolute"
            axis_xyz="1 0 0"
-           origin_rpy="0 0 0" origin_xyz="0 0 0.05"
+           origin_rpy="0 0 0" origin_xyz="0 0 0.058"
            parent="link_01" child="link_02"
            limit_e="1000" limit_l="-1.57" limit_u="1.57" limit_v="0.5" />
-  <m_link_mesh name="${link_02_name}"
+    <m_link_mesh name="${link_02_name}"
               origin_rpy="1.57 0 0" origin_xyz="0 0 -0.013"
               mass="157.633"
@@ -43,11 +43,11 @@
               meshfile="package://manipulator1ver/meshes/stl/3.stl"
               meshscale="0.001 0.001 0.001" />
-   <m_joint name="${link_02_name}__${link_03_name}" type="revolute"
+  <m_joint name="${link_02_name}__${link_03_name}" type="fixed"
            axis_xyz="1 0 0"
-           origin_rpy="0 0 0" origin_xyz="0 0.03 0.165"
+           origin_rpy="0 0 0" origin_xyz="0 0.0136 0.145"
            parent="link_02" child="link_03"
            limit_e="1000" limit_l="-1.57" limit_u="1.57" limit_v="0.5" />
-   <m_link_mesh name="${link_03_name}"
-              origin_rpy="0 0 0" origin_xyz="0 -0.013 0"
+    <m_link_mesh name="${link_03_name}"
+              origin_rpy="1.57 0 0" origin_xyz="0 0 0"
               mass="157.633"
               ixx="13.235" ixy="0" ixz="0"
@@ -56,11 +56,11 @@
               meshfile="package://manipulator1ver/meshes/stl/4.stl"
               meshscale="0.001 0.001 0.001" />
-   <m_joint name="${link_03_name}__${link_04_name}" type="revolute"
-           axis_xyz="0 1 0"
-           origin_rpy="0 0 0" origin_xyz="0 0 0"
+  <m_joint name="${link_03_name}__${link_04_name}" type="revolute"
+           axis_xyz="1 0 0"
+           origin_rpy="0 0 0" origin_xyz="0 0.017 0.0195"
            parent="link_03" child="link_04"
            limit_e="1000" limit_l="-1.57" limit_u="1.57" limit_v="0.5" />
-   <m_link_mesh name="${link_04_name}"
-              origin_rpy="0 3.14 0" origin_xyz="0 0.151 0"
+    <m_link_mesh name="${link_04_name}"
+              origin_rpy="1.57 0 0" origin_xyz="0 0.05 -0.0135"
               mass="157.633"
               ixx="13.235" ixy="0" ixz="0"
@@ -69,14 +69,11 @@
               meshfile="package://manipulator1ver/meshes/stl/5.stl"
               meshscale="0.001 0.001 0.001" />
-   <m_joint name="${link_04_name}__${link_05_name}" type="revolute"
+    <m_joint name="${link_04_name}__${link_05_name}" type="fixed"
            axis_xyz="1 0 0"
-           origin_rpy="0 0 0" origin_xyz="0.015 0.185 0"
+           origin_rpy="0 0 0" origin_xyz="0 0 0"
            parent="link_04" child="link_05"
            limit_e="1000" limit_l="-1.57" limit_u="1.57" limit_v="0.5" />
-<!--
-0 0.151 0
--->
-  <m_link_mesh name="${link_05_name}"
-              origin_rpy="1.57 -1.57 0" origin_xyz="0 0.056 0"
+    <m_link_mesh name="${link_05_name}"
+              origin_rpy="1.57 0 0" origin_xyz="0 0.13 -0.013"
               mass="157.633"
               ixx="13.235" ixy="0" ixz="0"
@@ -85,4 +82,45 @@
               meshfile="package://manipulator1ver/meshes/stl/6.stl"
               meshscale="0.001 0.001 0.001" />
+    <m_joint name="${link_05_name}__${link_06_name}" type="revolute"
+           axis_xyz="0 1 0"
+           origin_rpy="0 0 0" origin_xyz="0 0.185 0"
+           parent="link_05" child="link_06"
+           limit_e="1000" limit_l="-1.57" limit_u="1.57" limit_v="0.5" />
+    <m_link_mesh name="${link_06_name}"
+              origin_rpy="1.57 3.14 0" origin_xyz="0 -0.01 0.014"
+              mass="157.633"
+              ixx="13.235" ixy="0" ixz="0"
+              iyy="13.235" iyz="0"
+              izz="9.655"
+              meshfile="package://manipulator1ver/meshes/stl/7.stl"
+              meshscale="0.001 0.001 0.001" />
+  <m_joint name="${link_06_name}__${link_07_name}" type="revolute"
+           axis_xyz="1 0 0"
+           origin_rpy="0 0 0" origin_xyz="0 0 0"
+           parent="link_06" child="link_07"
+           limit_e="1000" limit_l="-1.57" limit_u="1.57" limit_v="0.5" />
+    <m_link_mesh name="${link_07_name}"
+              origin_rpy="1.57 3.14 0" origin_xyz="0 0.0175 0.02"
+              mass="157.633"
+              ixx="13.235" ixy="0" ixz="0"
+              iyy="13.235" iyz="0"
+              izz="9.655"
+              meshfile="package://manipulator1ver/meshes/stl/8.stl"
+              meshscale="0.001 0.001 0.001" />
+		<!--
+  <m_joint name="${link_07_name}__${link_08_name}" type="revolute"
+           axis_xyz="1 0 0"
+           origin_rpy="0 0 0" origin_xyz="0 0 0"
+           parent="link_07" child="link_08"
+           limit_e="1000" limit_l="-1.57" limit_u="1.57" limit_v="0.5" />
+    <m_link_mesh name="${link_08_name}"
+              origin_rpy="1.57 0 0" origin_xyz="0 0.0175 -0.02"
+              mass="157.633"
+              ixx="13.235" ixy="0" ixz="0"
+              iyy="13.235" iyz="0"
+              izz="9.655"
+              meshfile="package://manipulator1ver/meshes/stl/9.stl"
+              meshscale="0.001 0.001 0.001" />
+	-->
   <!-- END - Robot description -->
   <gazebo>

File: src/manipulator1ver/urdf/robot_parameters.xacro (robot description, xacro)
@@ -7,3 +7,6 @@
   <xacro:property name="link_04_name" value="link_04" />
   <xacro:property name="link_05_name" value="link_05" />
+  <xacro:property name="link_06_name" value="link_06" />
+  <xacro:property name="link_07_name" value="link_07" />
+  <xacro:property name="link_08_name" value="link_08" />
 </robot>

Commit message: RvizModelEnd

File: src/manipulator1ver/urdf/mrm.xacro (robot description, xacro)
@@ -2,5 +2,4 @@
 <robot name="mrm" xmlns:xacro="http://www.ros.org/wiki/xacro">
   <!-- BGN - Include -->
-  <xacro:include filename="$(find manipulator1ver)/urdf/robot_parameters.xacro" />
   <xacro:include filename="$(find manipulator1ver)/urdf/links_joints.xacro" />
   <!-- END - Include -->
@@ -9,5 +8,5 @@
   </material>
   <!-- BGN - Robot description -->
-  <m_link_mesh name="${link_00_name}"
+  <m_link_mesh name="link_00"
               origin_rpy="1.57 0 0" origin_xyz="0 0 0"
               mass="157.633"
@@ -15,12 +14,12 @@
               iyy="13.235" iyz="0"
               izz="9.655"
-              meshfile="package://manipulator1ver/meshes/stl/1base.stl"
+              meshfile="package://manipulator1ver/meshes/stlGrab/0ServoGrabBase.stl"
               meshscale="0.001 0.001 0.001" />
-  <m_joint name="${link_00_name}__${link_01_name}" type="revolute"
+  <m_joint name="Base" type="revolute"
            axis_xyz="0 0 1"
            origin_rpy="0 0 0" origin_xyz="0 0 0.0619"
-           parent="base_link" child="link_01"
+           parent="link_00" child="link_01"
            limit_e="1000" limit_l="-1.57" limit_u="1.57" limit_v="0.5" />
-  <m_link_mesh name="${link_01_name}"
+  <m_link_mesh name="link_01"
               origin_rpy="1.57 0 0" origin_xyz="0 0 0"
               mass="157.633"
@@ -28,12 +27,12 @@
               iyy="13.235" iyz="0"
               izz="9.655"
-              meshfile="package://manipulator1ver/meshes/stl/2.stl"
+              meshfile="package://manipulator1ver/meshes/stlGrab/1ServoGrab.stl"
               meshscale="0.001 0.001 0.001" />
-  <m_joint name="${link_01_name}__${link_02_name}" type="revolute"
+  <m_joint name="1stick" type="revolute"
            axis_xyz="1 0 0"
            origin_rpy="0 0 0" origin_xyz="0 0 0.058"
            parent="link_01" child="link_02"
            limit_e="1000" limit_l="-1.57" limit_u="1.57" limit_v="0.5" />
-    <m_link_mesh name="${link_02_name}"
+    <m_link_mesh name="link_02"
               origin_rpy="1.57 0 0" origin_xyz="0 0 -0.013"
               mass="157.633"
@@ -41,12 +40,39 @@
               iyy="13.235" iyz="0"
               izz="9.655"
-              meshfile="package://manipulator1ver/meshes/stl/3.stl"
+              meshfile="package://manipulator1ver/meshes/stlGrab/2ServoGrab.stl"
               meshscale="0.001 0.001 0.001" />
-  <m_joint name="${link_02_name}__${link_03_name}" type="fixed"
+  <m_joint name="2stick" type="revolute"
            axis_xyz="1 0 0"
-           origin_rpy="0 0 0" origin_xyz="0 0.0136 0.145"
+           origin_rpy="0 0 0" origin_xyz="0 0.0309 0.164"
            parent="link_02" child="link_03"
            limit_e="1000" limit_l="-1.57" limit_u="1.57" limit_v="0.5" />
-    <m_link_mesh name="${link_03_name}"
+    <m_link_mesh name="link_03"
+              origin_rpy="1.57 0 0" origin_xyz="0 -0.0139 -0.0203"
+              mass="157.633"
+              ixx="13.235" ixy="0" ixz="0"
+              iyy="13.235" iyz="0"
+              izz="9.655"
+              meshfile="package://manipulator1ver/meshes/stlGrab/3ServoGrab.stl"
+              meshscale="0.001 0.001 0.001" />
+  <m_joint name="3to4" type="revolute"
+           axis_xyz="1 0 0"
+           origin_rpy="0 0 0" origin_xyz="0  0.1597 0"
+           parent="link_03" child="link_04"
+           limit_e="1000" limit_l="-1.57" limit_u="1.57" limit_v="0.5" />
+    <m_link_mesh name="link_04"
+              origin_rpy="1.57 0 0" origin_xyz="0 -0.014 -0.014"
+              mass="157.633"
+              ixx="13.235" ixy="0" ixz="0"
+              iyy="13.235" iyz="0"
+              izz="9.655"
+              meshfile="package://manipulator1ver/meshes/stlGrab/4ServoGrab.stl"
+              meshscale="0.001 0.001 0.001" />
+<!-- GRAB -->
+  <m_joint name="GrabR" type="prismatic"
+           axis_xyz="1 0 0"
+           origin_rpy="0 0 0" origin_xyz="0.038 0.0855 -0.011"
+           parent="link_04" child="link_05"
+           limit_e="1000" limit_l="-0.02" limit_u="0" limit_v="0.5" />
+    <m_link_mesh name="link_05"
               origin_rpy="1.57 0 0" origin_xyz="0 0 0"
               mass="157.633"
@@ -54,73 +80,19 @@
               iyy="13.235" iyz="0"
               izz="9.655"
-              meshfile="package://manipulator1ver/meshes/stl/4.stl"
+              meshfile="package://manipulator1ver/meshes/stlGrab/5ServoGrab.stl"
               meshscale="0.001 0.001 0.001" />
-  <m_joint name="${link_03_name}__${link_04_name}" type="revolute"
+  <m_joint name="Grabl" type="prismatic"
            axis_xyz="1 0 0"
-           origin_rpy="0 0 0" origin_xyz="0 0.017 0.0195"
-           parent="link_03" child="link_04"
-           limit_e="1000" limit_l="-1.57" limit_u="1.57" limit_v="0.5" />
-    <m_link_mesh name="${link_04_name}"
-              origin_rpy="1.57 0 0" origin_xyz="0 0.05 -0.0135"
+           origin_rpy="0 0 0" origin_xyz="-0.038 0.0855 0.017"
+           parent="link_04" child="link_06"
+           limit_e="1000" limit_l="0" limit_u="0.02" limit_v="0.5" />
+    <m_link_mesh name="link_06"
+              origin_rpy="1.57 3.14 0" origin_xyz="0 0 0"
               mass="157.633"
               ixx="13.235" ixy="0" ixz="0"
               iyy="13.235" iyz="0"
               izz="9.655"
-              meshfile="package://manipulator1ver/meshes/stl/5.stl"
+              meshfile="package://manipulator1ver/meshes/stlGrab/5ServoGrab.stl"
               meshscale="0.001 0.001 0.001" />
-    <m_joint name="${link_04_name}__${link_05_name}" type="fixed"
-           axis_xyz="1 0 0"
-           origin_rpy="0 0 0" origin_xyz="0 0 0"
-           parent="link_04" child="link_05"
-           limit_e="1000" limit_l="-1.57" limit_u="1.57" limit_v="0.5" />
-    <m_link_mesh name="${link_05_name}"
-              origin_rpy="1.57 0 0" origin_xyz="0 0.13 -0.013"
-              mass="157.633"
-              ixx="13.235" ixy="0" ixz="0"
-              iyy="13.235" iyz="0"
-              izz="9.655"
-              meshfile="package://manipulator1ver/meshes/stl/6.stl"
-              meshscale="0.001 0.001 0.001" />
-    <m_joint name="${link_05_name}__${link_06_name}" type="revolute"
-           axis_xyz="0 1 0"
-           origin_rpy="0 0 0" origin_xyz="0 0.185 0"
-           parent="link_05" child="link_06"
-           limit_e="1000" limit_l="-1.57" limit_u="1.57" limit_v="0.5" />
-    <m_link_mesh name="${link_06_name}"
-              origin_rpy="1.57 3.14 0" origin_xyz="0 -0.01 0.014"
-              mass="157.633"
-              ixx="13.235" ixy="0" ixz="0"
-              iyy="13.235" iyz="0"
-              izz="9.655"
-              meshfile="package://manipulator1ver/meshes/stl/7.stl"
-              meshscale="0.001 0.001 0.001" />
-  <m_joint name="${link_06_name}__${link_07_name}" type="revolute"
-           axis_xyz="1 0 0"
-           origin_rpy="0 0 0" origin_xyz="0 0 0"
-           parent="link_06" child="link_07"
-           limit_e="1000" limit_l="-1.57" limit_u="1.57" limit_v="0.5" />
-    <m_link_mesh name="${link_07_name}"
-              origin_rpy="1.57 3.14 0" origin_xyz="0 0.0175 0.02"
-              mass="157.633"
-              ixx="13.235" ixy="0" ixz="0"
-              iyy="13.235" iyz="0"
-              izz="9.655"
-              meshfile="package://manipulator1ver/meshes/stl/8.stl"
-              meshscale="0.001 0.001 0.001" />
-		<!--
-  <m_joint name="${link_07_name}__${link_08_name}" type="revolute"
-           axis_xyz="1 0 0"
-           origin_rpy="0 0 0" origin_xyz="0 0 0"
-           parent="link_07" child="link_08"
-           limit_e="1000" limit_l="-1.57" limit_u="1.57" limit_v="0.5" />
-    <m_link_mesh name="${link_08_name}"
-              origin_rpy="1.57 0 0" origin_xyz="0 0.0175 -0.02"
-              mass="157.633"
-              ixx="13.235" ixy="0" ixz="0"
-              iyy="13.235" iyz="0"
-              izz="9.655"
-              meshfile="package://manipulator1ver/meshes/stl/9.stl"
-              meshscale="0.001 0.001 0.001" />
-	-->
   <!-- END - Robot description -->
   <gazebo>

File: src/manipulator1ver/urdf/robot_parameters.xacro (robot description, xacro)
@@ -1,12 +1,12 @@
 <?xml version="1.0" ?>
 <robot xmlns:xacro="http://www.ros.org/wiki/xacro">
-  <xacro:property name="link_00_name" value="base_link" />
-  <xacro:property name="link_01_name" value="link_01" />
-  <xacro:property name="link_02_name" value="link_02" />
-  <xacro:property name="link_03_name" value="link_03" />
-  <xacro:property name="link_04_name" value="link_04" />
-  <xacro:property name="link_05_name" value="link_05" />
-  <xacro:property name="link_06_name" value="link_06" />
-  <xacro:property name="link_07_name" value="link_07" />
-  <xacro:property name="link_08_name" value="link_08" />
+  <xacro:property name="link_00" value="0ServoGrabBase" />
+  <xacro:property name="link_01" value="1ServoGrab" />
+  <xacro:property name="link_02" value="2ServoGrab" />
+  <xacro:property name="link_03" value="3ServoGrab" />
+  <xacro:property name="link_04" value="4ServoGrab" />
+  <xacro:property name="link_05" value="5ServoGrab" />
+  <xacro:property name="link_06" value="link_06" />
+  <xacro:property name="link_07" value="link_07" />
+  <xacro:property name="link_08" value="link_08" />
 </robot>
